File: Robot_BMS/Solar.kicad_sch (KiCad schematic)
At the start: 19 parts, among them J3 691137710002, U5 LM3488MM, U9 CSD18563Q5A

Commit message: ex charging circuit last appearence
Parts:
- C23: renamed from C17; value 4n -> 990p
- C24: renamed from C18; value 240u -> 180n
- C25: renamed from C19; value 11p -> 820p
- R27: renamed from R23; value 12 -> 600
- R28: renamed from R24; value 47k5 -> 40k2
- R29: renamed from R25; value 8k -> 100
- R30: renamed from R26; value 3 milli_Ohm -> 13 milli_Ohm
- renumbered C15 to C21, C16 to C22, C20 to C26, C21 to C27, D2 to D1, R22 to R26, R27 to R31, R28 to R32, U9 to U6
Connections:
- net SOLAR_13V_OUT renamed SOLAR_15V_OUT
Other:
- note added: "Common Solar panels can produce anything from 28V to 4V. We want to feed a 15V output to our Li Ion chargers. Uses a sepic dc/dc converter"
- note removed: "Common Solar panels can produce anything from 28V to 4V. We want to feed a 13V output to our Li Ion chargers. Uses a sepic dc/dc converter"
Changed lines of the file:
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@@
 		)
 	)
-	(text "Common Solar panels can produce anything\nfrom 28V to 4V. We want to feed a 13V output \nto our Li Ion chargers.\nUses a sepic dc/dc converter"
+	(text "Common Solar panels can produce anything\nfrom 28V to 4V. We want to feed a 15V output \nto our Li Ion chargers.\nUses a sepic dc/dc converter"
 		(exclude_from_sim no)
 		(at 237.49 23.114 0)
@@
 		)
 	)
-	(hierarchical_label "SOLAR_13V_OUT"
+	(hierarchical_label "SOLAR_15V_OUT"
 		(shape output)
 		(at 261.874 53.086 0)
@@
 		(on_board yes)
 		(dnp no)
-		(property "Reference" "#PWR026"
+		(property "Reference" "#PWR037"
 			(at 60.452 112.776 0)
 			(effects
@@
 			(project "Robot_BMS"
 				(path "/72551b1c-3d40-4199-8911-e5b015f4abec/ff8c01d9-7d3c-4161-8f4f-7a8402a9daec"
-					(reference "#PWR026")
+					(reference "#PWR037")
 					(unit 1)
 				)
@@
 		(on_board yes)
 		(dnp no)
-		(property "Reference" "#PWR033"
+		(property "Reference" "#PWR044"
 			(at 161.544 105.664 0)
 			(effects
@@
 			(project "Robot_BMS"
 				(path "/72551b1c-3d40-4199-8911-e5b015f4abec/ff8c01d9-7d3c-4161-8f4f-7a8402a9daec"
-					(reference "#PWR033")
+					(reference "#PWR044")
 					(unit 1)
 				)
@@
 		(dnp no)
 		(fields_autoplaced yes)
-		(property "Reference" "C15"
+		(property "Reference" "C21"
 			(at 48.26 80.0099 0)
 			(effects
@@
 			(project ""
 				(path "/72551b1c-3d40-4199-8911-e5b015f4abec/ff8c01d9-7d3c-4161-8f4f-7a8402a9daec"
-					(reference "C15")
+					(reference "C21")
 					(unit 1)
 				)
@@
 		(on_board yes)
 		(dnp no)
-		(property "Reference" "U9"
+		(property "Reference" "U6"
 			(at 214.63 85.09 90)
 			(effects
@@
 			(project ""
 				(path "/72551b1c-3d40-4199-8911-e5b015f4abec/ff8c01d9-7d3c-4161-8f4f-7a8402a9daec"
-					(reference "U9")
+					(reference "U6")
 					(unit 1)
 				)
@@
 		(dnp no)
 		(fields_autoplaced yes)
-		(property "Reference" "D2"
+		(property "Reference" "D1"
 			(at 210.312 43.688 0)
 			(effects
@@
 			(project ""
 				(path "/72551b1c-3d40-4199-8911-e5b015f4abec/ff8c01d9-7d3c-4161-8f4f-7a8402a9daec"
-					(reference "D2")
+					(reference "D1")
 					(unit 1)
 				)
@@
 		(dnp no)
 		(fields_autoplaced yes)
-		(property "Reference" "R23"
+		(property "Reference" "R27"
 			(at 90.17 67.0559 0)
 			(effects
@@
 			)
 		)
-		(property "Value" "12"
+		(property "Value" "600"
 			(at 90.17 69.5959 0)
 			(effects
@@
 			(project "Robot_BMS"
 				(path "/72551b1c-3d40-4199-8911-e5b015f4abec/ff8c01d9-7d3c-4161-8f4f-7a8402a9daec"
-					(reference "R23")
+					(reference "R27")
 					(unit 1)
 				)
@@
 		(on_board yes)
 		(dnp no)
-		(property "Reference" "#PWR030"
+		(property "Reference" "#PWR041"
 			(at 99.06 90.17 0)
 			(effects
@@
 			(project "Robot_BMS"
 				(path "/72551b1c-3d40-4199-8911-e5b015f4abec/ff8c01d9-7d3c-4161-8f4f-7a8402a9daec"
-					(reference "#PWR030")
+					(reference "#PWR041")
 					(unit 1)
 				)
@@
 		(dnp no)
 		(fields_autoplaced yes)
-		(property "Reference" "R25"
+		(property "Reference" "R29"
 			(at 105.41 125.73 90)
 			(effects
@@
 			)
 		)
-		(property "Value" "8k"
+		(property "Value" "100"
 			(at 105.41 128.27 90)
 			(effects
@@
 			(project "Robot_BMS"
 				(path "/72551b1c-3d40-4199-8911-e5b015f4abec/ff8c01d9-7d3c-4161-8f4f-7a8402a9daec"
-					(reference "R25")
+					(reference "R29")
 					(unit 1)
 				)
@@
 		(dnp no)
 		(fields_autoplaced yes)
-		(property "Reference" "R26"
+		(property "Reference" "R30"
 			(at 119.38 141.4779 0)
 			(effects
@@
 			)
 		)
-		(property "Value" "3 milli_Ohm"
+		(property "Value" "13 milli_Ohm"
 			(at 119.38 144.0179 0)
 			(effects
@@
 			(project "Robot_BMS"
 				(path "/72551b1c-3d40-4199-8911-e5b015f4abec/ff8c01d9-7d3c-4161-8f4f-7a8402a9daec"
-					(reference "R26")
+					(reference "R30")
 					(unit 1)
 				)
@@
 		(dnp no)
 		(fields_autoplaced yes)
-		(property "Reference" "R24"
+		(property "Reference" "R28"
 			(at 101.6 76.1999 0)
 			(effects
@@
 			)
 		)
-		(property "Value" "47k5"
+		(property "Value" "40k2"
 			(at 101.6 78.7399 0)
 			(effects
@@
 			(project ""
 				(path "/72551b1c-3d40-4199-8911-e5b015f4abec/ff8c01d9-7d3c-4161-8f4f-7a8402a9daec"
-					(reference "R24")
+					(reference "R28")
 					(unit 1)
 				)
@@
 		(dnp no)
 		(fields_autoplaced yes)
-		(property "Reference" "C21"
+		(property "Reference" "C27"
 			(at 251.46 67.5639 0)
 			(effects
@@
 			(project "Robot_BMS"
 				(path "/72551b1c-3d40-4199-8911-e5b015f4abec/ff8c01d9-7d3c-4161-8f4f-7a8402a9daec"
-					(reference "C21")
+					(reference "C27")
 					(unit 1)
 				)
@@
 		(dnp no)
 		(fields_autoplaced yes)
-		(property "Reference" "R28"
+		(property "Reference" "R32"
 			(at 228.6 76.1999 0)
 			(effects
@@
 			(project "Robot_BMS"
 				(path "/72551b1c-3d40-4199-8911-e5b015f4abec/ff8c01d9-7d3c-4161-8f4f-7a8402a9daec"
-					(reference "R28")
+					(reference "R32")
 					(unit 1)
 				)
@@
 		(on_board yes)
 		(dnp no)
-		(property "Reference" "#PWR034"
+		(property "Reference" "#PWR045"
 			(at 248.412 99.568 0)
 			(effects
@@
 			(project "Robot_BMS"
 				(path "/72551b1c-3d40-4199-8911-e5b015f4abec/ff8c01d9-7d3c-4161-8f4f-7a8402a9daec"
-					(reference "#PWR034")
+					(reference "#PWR045")
 					(unit 1)
 				)
@@
 		(on_board yes)
 		(dnp no)
-		(property "Reference" "C20"
+		(property "Reference" "C26"
 			(at 185.166 45.466 90)
 			(effects
@@
 			(project "Robot_BMS"
 				(path "/72551b1c-3d40-4199-8911-e5b015f4abec/ff8c01d9-7d3c-4161-8f4f-7a8402a9daec"
-					(reference "C20")
+					(reference "C26")
 					(unit 1)
 				)
@@
 		(on_board yes)
 		(dnp no)
-		(property "Reference" "#PWR027"
+		(property "Reference" "#PWR038"
 			(at 74.422 91.694 0)
 			(effects
@@
 			(project "Robot_BMS"
 				(path "/72551b1c-3d40-4199-8911-e5b015f4abec/ff8c01d9-7d3c-4161-8f4f-7a8402a9daec"
-					(reference "#PWR027")
+					(reference "#PWR038")
 					(unit 1)
 				)
@@
 		(on_board yes)
 		(dnp no)
-		(property "Reference" "#PWR028"
+		(property "Reference" "#PWR039"
 			(at 87.63 92.202 0)
 			(effects
@@
 			(project "Robot_BMS"
 				(path "/72551b1c-3d40-4199-8911-e5b015f4abec/ff8c01d9-7d3c-4161-8f4f-7a8402a9daec"
-					(reference "#PWR028")
+					(reference "#PWR039")
 					(unit 1)
 				)
@@
 		(dnp no)
 		(fields_autoplaced yes)
-		(property "Reference" "R22"
+		(property "Reference" "R26"
 			(at 62.23 71.8819 0)
 			(effects
@@
 			(project ""
 				(path "/72551b1c-3d40-4199-8911-e5b015f4abec/ff8c01d9-7d3c-4161-8f4f-7a8402a9daec"
-					(reference "R22")
+					(reference "R26")
 					(unit 1)
 				)
@@
 		(dnp no)
 		(fields_autoplaced yes)
-		(property "Reference" "C18"
+		(property "Reference" "C24"
 			(at 91.44 77.7239 0)
 			(effects
@@
 			)
 		)
-		(property "Value" "240u"
+		(property "Value" "180n"
 			(at 91.44 80.2639 0)
 			(effects
@@
 			(project "Robot_BMS"
 				(path "/72551b1c-3d40-4199-8911-e5b015f4abec/ff8c01d9-7d3c-4161-8f4f-7a8402a9daec"
-					(reference "C18")
+					(reference "C24")
 					(unit 1)
 				)
@@
 		(dnp no)
 		(fields_autoplaced yes)
-		(property "Reference" "C16"
+		(property "Reference" "C22"
 			(at 63.5 96.7739 0)
 			(effects
@@
 			(project "Robot_BMS"
 				(path "/72551b1c-3d40-4199-8911-e5b015f4abec/ff8c01d9-7d3c-4161-8f4f-7a8402a9daec"
-					(reference "C16")
+					(reference "C22")
 					(unit 1)
 				)
@@
 		(on_board yes)
 		(dnp no)
-		(property "Reference" "#PWR032"
+		(property "Reference" "#PWR042"
 			(at 116.84 53.086 0)
 			(effects
@@
 			(project "Robot_BMS"
 				(path "/72551b1c-3d40-4199-8911-e5b015f4abec/ff8c01d9-7d3c-4161-8f4f-7a8402a9daec"
-					(reference "#PWR032")
+					(reference "#PWR042")
 					(unit 1)
 				)
@@
 		(on_board yes)
 		(dnp no)
-		(property "Reference" "#PWR031"
+		(property "Reference" "#PWR043"
 			(at 116.84 157.734 0)
 			(effects
@@
 			(project "Robot_BMS"
 				(path "/72551b1c-3d40-4199-8911-e5b015f4abec/ff8c01d9-7d3c-4161-8f4f-7a8402a9daec"
-					(reference "#PWR031")
+					(reference "#PWR043")
 					(unit 1)
 				)
@@
 		(dnp no)
 		(fields_autoplaced yes)
-		(property "Reference" "C19"
+		(property "Reference" "C25"
 			(at 97.79 142.2399 0)
 			(effects
@@
 			)
 		)
-		(property "Value" "11p"
+		(property "Value" "820p"
 			(at 97.79 144.7799 0)
 			(effects
@@
 			(project "Robot_BMS"
 				(path "/72551b1c-3d40-4199-8911-e5b015f4abec/ff8c01d9-7d3c-4161-8f4f-7a8402a9daec"
-					(reference "C19")
+					(reference "C25")
 					(unit 1)
 				)
@@
 		(on_board yes)
 		(dnp no)
-		(property "Reference" "#PWR029"
+		(property "Reference" "#PWR040"
 			(at 94.234 157.734 0)
 			(effects
@@
 			(project "Robot_BMS"
 				(path "/72551b1c-3d40-4199-8911-e5b015f4abec/ff8c01d9-7d3c-4161-8f4f-7a8402a9daec"
-					(reference "#PWR029")
+					(reference "#PWR040")
 					(unit 1)
 				)
@@
 		(dnp no)
 		(fields_autoplaced yes)
-		(property "Reference" "C17"
+		(property "Reference" "C23"
 			(at 77.47 76.9619 0)
 			(effects
@@
 			)
 		)
-		(property "Value" "4n"
+		(property "Value" "990p"
 			(at 77.47 79.5019 0)
 			(effects
@@
 			(project "Robot_BMS"
 				(path "/72551b1c-3d40-4199-8911-e5b015f4abec/ff8c01d9-7d3c-4161-8f4f-7a8402a9daec"
-					(reference "C17")
+					(reference "C23")
 					(unit 1)
 				)
@@
 		(dnp no)
 		(fields_autoplaced yes)
-		(property "Reference" "R27"
+		(property "Reference" "R31"
 			(at 228.6 58.6739 0)
 			(effects
@@
 			(project "Robot_BMS"
 				(path "/72551b1c-3d40-4199-8911-e5b015f4abec/ff8c01d9-7d3c-4161-8f4f-7a8402a9daec"
-					(reference "R27")
-					(unit 1)
-				)
+					(reference "R31")
+					(unit 1)
+				)
